File: pcb/ESP32-Mini-Matrix-Shield-DMA.brd (EAGLE design)
At the start: 68.2 x 54.6 mm, 29 parts, among them J1 5.5/2.1mm, P1 M-2X08-DIL-100

Commit message: Updated PCB to v0.3
Parts:
- added D1': 20V-1A, OPL_Discrete_Semiconductor:SOD-123
- added JTAG: M-2X05-DIL-100, con-headers-jp:DIL-100-2X05
- added PROG: M-2X03-DIL-100, con-headers-jp:DIL-100-2X03
- D1: value 20V-1A -> Schottky; device OPL_Discrete_Semiconductor:SOD-123 -> diode:DO41-10
- moved J1 45.8 mm to (59.7, 12.7), turned to 90 degrees
- moved JP1 39.4 mm to (53.1, 13.5), turned to 0 degrees
- moved D1 22.9 mm to (48.3, 12.7), flipped to the top, turned to 270 degrees
- moved ST_01 14.0 mm to (34.3, 10.2)
- moved 5V_T 11.5 mm to (24.1, 5.08)
- moved GND_T 11.5 mm to (14.0, 5.08)
- moved ESP32_D1_MINI 6.84 mm to (48.3, 27.9)
- moved P1 5.68 mm to (34.3, 38.1)
- moved E_SEL 4.58 mm to (39.4, 34.3)
- moved R2 2.84 mm to (58.4, 44.5)
- moved R2' 2.84 mm to (58.7, 44.5)
- moved I2C_VCC_SEL 2.84 mm to (58.4, 22.9)
- moved R1 2.84 mm to (58.4, 31.8)
- moved R1' 2.84 mm to (58.7, 31.8)
- moved H1 1.27 mm to (64.8, 3.81)
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Connections:
- removed net B2: ESP32_D1_MINI.TCK, P1.7
- removed net G2: ESP32_D1_MINI.TDI, P1.6
- removed net OE: ESP32_D1_MINI.TD0, P1.14
- removed net R2: ESP32_D1_MINI.TMS, P1.5
- new net ESP_IO0: ESP32_D1_MINI.IO0, PROG.6
- new net ESP_RXD: ESP32_D1_MINI.RXD, PROG.5
- new net ESP_TXD: ESP32_D1_MINI.TXD, PROG.3
- new net NC3: JTAG.10
- new net RST: ESP32_D1_MINI.RST, PROG.1
- new net TCK: ESP32_D1_MINI.TCK, JTAG.4, P1.7
- new net TDI: ESP32_D1_MINI.TDI, JTAG.8, P1.6
- new net TDO: ESP32_D1_MINI.TD0, JTAG.6, P1.15
- new net TMS: ESP32_D1_MINI.TMS, JTAG.2, P1.5
- net 3V3: now also JTAG.1, PROG.2
- net 5V: now also D1'.-, D1.C; no longer D1.-
- net 5V_EXT: now also D1'.+, D1.A; no longer D1.+
- net GND: now also JTAG.3, JTAG.5, JTAG.7, JTAG.9, PROG.4
- net LS: now also P1.14; no longer P1.15
Routing:
- net TDI: track 0.00 -> 61.6 mm
- net ESP_TXD: track 0.00 -> 43.7 mm
- net TDO: track 0.00 -> 42.7 mm
- net TMS: track 0.00 -> 42.2 mm, vias 0 -> 1
- net ESP_RXD: track 0.00 -> 41.6 mm
- net TCK: track 0.00 -> 37.8 mm
- net RST: track 0.00 -> 33.3 mm, vias 0 -> 1
- net IO32: track 55.0 -> 85.2 mm, vias 1 -> 0
- net ESP_IO0: track 0.00 -> 24.5 mm, vias 0 -> 1
- net SCL: track 88.2 -> 110.7 mm
- net 3V3: track 56.2 -> 74.6 mm, vias 1 -> 2
- net 5V: track 64.4 -> 81.2 mm
- net R2: track 16.2 -> 0.00 mm
- net IO35: track 32.1 -> 16.3 mm
- net B2: track 14.4 -> 0.00 mm, vias 1 -> 0
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Other:
- board text added: "ESP32 Matrix DMA Shield v0.3 http://github.com/bogd"
- board text added: "I2C_1"
- board text added: "I2C_2"
- board text added: "I2C_3"
- board text added: "I2C_4"
- board text added: "Mount D1 Mini on other side of the board, metal plate this way!"
- board text removed: "ESP32 Matrix DMA Shield v0.1 http://github.com/bogd"
- board text removed: "Mount on other side of the board, metal plate facing this way!"
