File: pcb/ESP32-Mini-Matrix-Shield-DMA.sch (EAGLE design)
At the start: 29 parts, among them J1 5.5/2.1mm, P1 M-2X08-DIL-100

Commit message: Updated PCB to v0.3
Parts:
- added D1': 20V-1A, OPL_Discrete_Semiconductor:SMD-DIODE-SCHOTTKY-20V-1A(SOD-123)
- added JTAG: M-2X05-DIL-100, con-headers-jp:M-2X05-DIL-100
- added PROG: M-2X03-DIL-100, con-headers-jp:M-2X03-DIL-100
- D1: value 20V-1A -> Schottky; device OPL_Discrete_Semiconductor:SMD-DIODE-SCHOTTKY-20V-1A(SOD-123) -> diode:1N4004
Connections:
- removed net B2: ESP32_D1_MINI.TCK, P1.7
- removed net G2: ESP32_D1_MINI.TDI, P1.6
- removed net OE: ESP32_D1_MINI.TD0, P1.14
- removed net R2: ESP32_D1_MINI.TMS, P1.5
- new net ESP_IO0: ESP32_D1_MINI.IO0, PROG.6
- new net ESP_RXD: ESP32_D1_MINI.RXD, PROG.5
- new net ESP_TXD: ESP32_D1_MINI.TXD, PROG.3
- new net NC3: JTAG.10
- new net RST: ESP32_D1_MINI.RST, PROG.1
- new net TCK: ESP32_D1_MINI.TCK, JTAG.4, P1.7
- new net TDI: ESP32_D1_MINI.TDI, JTAG.8, P1.6
- new net TDO: ESP32_D1_MINI.TD0, JTAG.6, P1.15
- new net TMS: ESP32_D1_MINI.TMS, JTAG.2, P1.5
- net 3V3: now also JTAG.1, PROG.2
- net 5V: now also D1'.-, D1.C; no longer D1.-
- net 5V_EXT: now also D1'.+, D1.A; no longer D1.+
- net GND: now also JTAG.3, JTAG.5, JTAG.7, JTAG.9, PROG.4
- net LS: now also P1.14; no longer P1.15
Other:
- moved on the sheet: E_SEL, GND_T-1, GND_T-2, P1
